Commit message: Add reset function

File: tests/urdf/hole_round.urdf (robot description, URDF)
Before this commit: robot hole_round, 1 links, 0 joints
Links:
- added link hole_target_link, mass 0
Joints:
- added joint hole_link-hole_target_link: type fixed, parent hole_link, child hole_target_link, origin xyz=0.0 0.0 0.0 rpy=0.0 0.0 0.0

File: tests/urdf/peg_round.urdf (robot description, URDF)
Before this commit: robot peg_round, 1 links, 0 joints
Links:
- added link peg_target_link, mass 0
Joints:
- added joint peg_link-peg_target_link: type fixed, parent peg_link, child peg_target_link, origin xyz=0.0 0.0 0.0 rpy=0.0 0.0 0.0
