Commit message: Add Env with peg in hole task Configure reward and observation for peg

File: tests/urdf/peg_round.urdf (robot description, URDF)
Before this commit: robot peg_round, 2 links, 1 joints
Joints:
- joint peg_link-peg_target_link: origin xyz=0.0 0.0 0.0 rpy=0.0 0.0 0.0 -> xyz=0.0 0.0 0.052 rpy=0.0 0.0 0.0
