Commit message: add egg into egg

File: tests/urdf/peg_sqr.urdf (robot description, URDF)
Before this commit: robot peg_round, 2 links, 1 joints
Links:
- link peg_link: geometry collision mesh filename=meshes/peg/peg_sqr.STL scale=0.001 0.001 0.001; visual mesh filename=meshes/peg/peg_sqr.STL scale=0.001 0.001 0.001

File: tests/urdf/ur5e_pybullet.urdf (robot description, URDF)
Before this commit: robot ur5e, 12 links, 11 joints
Links:
- added link camera_link, mass 0
Joints:
- added joint camera_link_joint: type fixed, parent tool0, child camera_link, origin xyz=0.00 -0.08 0.0 rpy=-0.1 0.0 0.0
