Commit message: Add resource files

File: src/itmobotics_gym/envs/models/hole_round.urdf (robot description, URDF)
Before this commit: robot hole_round, 1 links, 0 joints
Links:
- added link hole_target_link, mass 0
Joints:
- added joint hole_link-hole_target_link: type fixed, parent hole_link, child hole_target_link, origin xyz=0.0 0.0 0.0 rpy=0.0 0.0 0.0

File: src/itmobotics_gym/envs/models/hole_sqr.urdf (robot description, URDF)
Before this commit: robot hole_sqr, 1 links, 0 joints
Links:
- added link hole_target_link, mass 0
Joints:
- added joint hole_link-hole_target_link: type fixed, parent hole_link, child hole_target_link, origin xyz=0.0 0.0 0.0 rpy=0.0 0.0 0.0
